Commit message: a bit of video recording

File: src/racecar.xacro (robot description, xacro)
@@ -21,5 +21,5 @@
       <origin xyz="${wheelbase/2} 0 ${ground_offset+height/2}"/>
       <geometry>
-        <box size="${wheelbase} ${width} ${height}"/>
+        <box size="${wheelbase*2} ${width*2} ${height}"/>
       </geometry>
       <material name="red"/>
